File: Small/Small.kicad_pcb (KiCad board)
At the start: 2 copper layers, 120 x 103.9 mm, 93 parts, among them J1 Conn_Ext_0, J10 Conn_01x03_Female, J11 Conn_01x03_Female, J12 Conn_01x03_Female, J13 Conn_01x03_Female, J14 Conn_01x03_Female, J15 Conn_01x03_Female, J16 Conn_01x03_Female, J17 Conn_01x03_Female, J18 Conn_01x03_Female, J19 Conn_01x03_Female, J2 Conn_Alt_0, J20 Conn_01x03_Female, J21 Conn_01x03_Female, J22 Conn_01x03_Female, J23 Conn_01x03_Female, J24 Conn_01x03_Female, J25 Conn_01x03_Female, J27 SWD_TAG_Connector, J3 Conn_Ext_4, J4 Conn_Alt_4, J5 Conn_Ext_8, J6 Conn_SWD, J7 Conn_Alt_8, J8 Conn_01x03_Female, J9 Conn_01x03_Female, Q1 NMOS, Q2 NMOS, Q3 NMOS, Q4 NMOS, Q5 NMOS, Q6 NMOS, SW1 SW_Push, U1 TLVM23625RDNR, U2 STM32G070KBT6, U3 AP7361C-33E, U4 TXB0102DCU, Y1 Crystal_GND24

Commit message: [SMA] Improve PCB
Parts:
- removed the R21 at (273.4, 63.6)
- removed R22: 10k, Resistor_SMD:R_0805_2012Metric_Pad1.20x1.40mm_HandSolder
- removed the R25 at (278.1, 54.8)
- removed R26: 0, Resistor_SMD:R_0805_2012Metric_Pad1.20x1.40mm_HandSolder
- D1, D2, D3, D4, D5, D6, J27: moved to B.Cu
- J2: moved to F.Cu
- moved D6 241.9 mm to (47.5, 70.9), turned to 150 degrees
- moved D5 240.7 mm to (48.8, 68.8), turned to 150 degrees
- moved R24 233.1 mm to (46.7, 79.7), turned to -120 degrees
- moved C11 230.5 mm to (65.3, 68.4), turned to 60 degrees
- moved R18 229.6 mm to (49.5, 105.7), turned to -60 degrees
- moved R20 229.3 mm to (44.8, 77.5), turned to 150 degrees
- moved R17 224.0 mm to (51.5, 82.4), turned to 60 degrees
- moved R23 221.2 mm to (57.5, 64.6), turned to 60 degrees
- moved R16 221.0 mm to (52.8, 61.8), turned to -120 degrees
- moved C14 220.4 mm to (75.0, 79.1), turned to 180 degrees
- moved J14 219.2 mm to (47.5, 113.2), turned to 180 degrees
- moved C15 218.2 mm to (74.8, 72.1), turned to 180 degrees
- moved R19 214.1 mm to (59.5, 66.8), turned to -30 degrees
- moved J19 213.7 mm to (34.6, 99.6), turned to 60 degrees
- moved C13 212.5 mm to (75.0, 77.0), turned to 180 degrees
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Routing:
- net VDD: track 0.00 -> 168.8 mm
- net GND: track 0.00 -> 118.9 mm, vias 0 -> 2
- net +5V: track 0.00 -> 67.1 mm
- net Net-(J10-Pin_2): track 0.00 -> 44.0 mm
- net Net-(J11-Pin_2): track 0.00 -> 43.0 mm
- net /UART_3_RX: track 0.00 -> 35.3 mm
- net /UART_2_RX: track 0.00 -> 34.7 mm
- net /UART_1_RX: track 0.00 -> 34.5 mm
- net /NRST: track 0.00 -> 32.6 mm, vias 0 -> 2
- net /UART_3_TX: track 0.00 -> 28.2 mm
- net /UART_1_TX: track 0.00 -> 26.3 mm
- net Net-(J13-Pin_2): track 0.00 -> 25.7 mm
- net Net-(J14-Pin_2): track 0.00 -> 24.6 mm
- net /UART_2_TX: track 0.00 -> 13.6 mm
- net +3V3: track 0.00 -> 12.5 mm
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Other:
- outline, holes or cut-outs redrawn

Commit message: [SMA] Finish PCB
Parts:
- C12, C16, R15, Y1: moved to B.Cu
- moved C9 88.7 mm to (51.8, 89.7), turned to 30 degrees
- moved U3 86.2 mm to (56.3, 92.5), turned to 30 degrees
- moved C10 83.9 mm to (56.4, 97.8), turned to 30 degrees
- moved C16 57.6 mm to (73.0, 91.1)
- moved C12 54.9 mm to (75.8, 88.7), turned to 90 degrees
- moved Y1 54.9 mm to (73.5, 88.7), turned to 90 degrees
- moved R15 54.4 mm to (71.2, 88.2), turned to 90 degrees
Connections:
- U1 pad 10: (no net) -> GND
Routing:
- net +5V: track 67.1 -> 432.8 mm, vias 0 -> 6
- net GND: track 118.9 -> 271.8 mm, vias 2 -> 31
- net +3V3: track 12.5 -> 125.1 mm, vias 0 -> 7
- net /SWDIO: track 0.00 -> 59.0 mm, vias 0 -> 5
- net /SWDCLK: track 0.00 -> 53.6 mm, vias 0 -> 3
- net /LED_RET: track 0.00 -> 34.8 mm, vias 0 -> 2
- net /LED_SIG: track 0.00 -> 33.9 mm, vias 0 -> 2
- net /UART_2_TX: track 13.6 -> 45.2 mm, vias 0 -> 3
- net Net-(D2-A): track 0.00 -> 14.7 mm, vias 0 -> 1
- net /NRST: track 32.6 -> 47.1 mm, vias 2 -> 3
- net Net-(D6-A): track 0.00 -> 13.4 mm, vias 0 -> 1
- net Net-(D4-A): track 0.00 -> 12.8 mm, vias 0 -> 1
- net Net-(D4-K): track 0.00 -> 11.8 mm, vias 0 -> 1
- net Net-(D2-K): track 0.00 -> 11.7 mm, vias 0 -> 1
- net Net-(D6-K): track 0.00 -> 11.4 mm, vias 0 -> 1
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- added copper zone on B.Cu, net GND
- added copper zone on F.Cu, net GND

Commit message: [SMA] Fix many  bug
Parts:
- moved H2 100.3 mm to (28.7, 115.0)
- moved H1 97.7 mm to (121.3, 115.0)
- moved H3 95.3 mm to (75.0, 34.7)
- moved J11 15.1 mm to (87.3, 52.3)
- moved J12 15.1 mm to (65.2, 47.9)
- moved C13 14.5 mm to (66.7, 89.0), turned to -90 degrees
- moved J17 13.9 mm to (84.5, 57.0)
- moved J18 13.4 mm to (63.1, 61.0)
- moved J23 13.2 mm to (91.1, 55.8)
- moved J24 13.2 mm to (58.9, 55.8)
- moved J8 12.7 mm to (45.0, 116.9)
- moved J9 12.7 mm to (100.0, 116.9)
- moved C14 11.7 mm to (68.8, 89.0), turned to -90 degrees
- moved C15 10.7 mm to (81.8, 64.0), turned to -90 degrees
- moved J10 10.2 mm to (114.8, 99.9)
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Connections:
- U2 pad 1: /UART_2_RX -> unconnected-(U2-PB9-Pad1)
- U2 pad 10: unconnected-(U2-PA3-Pad10) -> /UART_1_RX
- U2 pad 12: /UART_2_TX -> unconnected-(U2-PA5-Pad12)
- U2 pad 19: /UART_1_TX -> /UART_2_TX
- U2 pad 21: /UART_1_RX -> /UART_2_RX
- U2 pad 9: unconnected-(U2-PA2-Pad9) -> /UART_1_TX
Routing:
- net GND: track 271.8 -> 184.4 mm, vias 31 -> 27
- net +5V: track 432.8 -> 395.5 mm, vias 6 -> 7
- net +3V3: track 125.1 -> 94.5 mm, vias 7 -> 4
- net Net-(J11-Pin_2): track 43.0 -> 64.4 mm
- net /NRST: track 47.1 -> 61.1 mm, vias 3 -> 5
- net /UART_3_TX: track 37.4 -> 48.0 mm, vias 1 -> 0
- net /SWDIO: track 59.0 -> 53.0 mm, vias 5 -> 2
- net /UART_1_TX: track 35.4 -> 41.0 mm, vias 1 -> 0
- net /OSC_OUT: track 10.2 -> 5.20 mm
- net /SWDCLK: track 53.6 -> 48.7 mm, vias 3 -> 1
- net Net-(J13-Pin_2): track 25.9 -> 30.7 mm
- net /OSC_IN: track 8.93 -> 5.07 mm
- net /UART_2_TX: track 45.2 -> 41.7 mm, vias 3 -> 0
- net VDD: track 168.8 -> 165.4 mm
- net /LED_SIG: track 33.9 -> 37.3 mm, vias 2 -> 4
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Other:
- board size 120 x 103.9 mm -> 110 x 95.3 mm
