File: Small/Small.kicad_sch (KiCad schematic)
At the start: 34 parts, among them J1 Conn_SWD, J2 Conn_01x03_Female, J3 Conn_01x03_Female, J4 Conn_01x03_Female, J5 Conn_01x03_Female, J6 Conn_01x03_Female, J7 Conn_01x03_Female, SW1 SW_Push, U1 STM32G070KBT6, U2 AP7361C-33E, U3 TPS54331DR, Y1 Crystal

Commit message: [SMA] Improve schematic
Parts:
- added C14, C15, C16: C, symbol Device:C
- added D2, D3, D4, D5, D6, D7: LED, LED_SMD:LED_0805_2012Metric_Pad1.15x1.40mm_HandSolder, symbol Device:LED
- added J10: Conn_Ext_8, symbol Connector_Generic:Conn_01x04
- added J8: Conn_Ext_0, symbol Connector_Generic:Conn_01x04
- added J9: Conn_Ext_4, symbol Connector_Generic:Conn_01x04
- added Q1: Q_PMOS_DGS, symbol Device:Q_PMOS_DGS
- added Q2, Q3, Q4, Q5, Q6, Q7: NMOS, symbol Device:Q_NMOS_DGS
- added R10, R13, R16, R21, R22, R27, R9: 0, Resistor_SMD:R_0805_2012Metric_Pad1.20x1.40mm_HandSolder, symbol Device:R
- added R11, R14, R17, R20, R23, R26, R8: 10k, Resistor_SMD:R_0805_2012Metric_Pad1.20x1.40mm_HandSolder, symbol Device:R
- added R12, R15, R18, R19, R24, R25: R, Resistor_SMD:R_0805_2012Metric_Pad1.20x1.40mm_HandSolder, symbol Device:R
- C1, C10, C11, C12, C2, C3, C6, C7, C9: footprint (none) -> Capacitor_SMD:C_0805_2012Metric_Pad1.18x1.45mm_HandSolder
- C13: footprint (none) -> Capacitor_SMD:CP_Elec_5x3
- C4, C5: value TBD -> DNP; footprint (none) -> Capacitor_SMD:C_0805_2012Metric_Pad1.18x1.45mm_HandSolder
- J2, J3, J4, J5, J6, J7: footprint (none) -> Connector_JST:JST_XH_B3B-XH-A_1x03_P2.50mm_Vertical
- R1: value TBD -> DNP; footprint (none) -> Resistor_SMD:R_0805_2012Metric_Pad1.20x1.40mm_HandSolder
- R2, R3, R4, R5, R6, R7: footprint (none) -> Resistor_SMD:R_0805_2012Metric_Pad1.20x1.40mm_HandSolder
Connections:
- net +5V: now also Q1.1 (D), R12.1, R15.1, R18.1, R19.1, R24.1, R25.1
- net GND: now also C14.2, C15.2, C16.2, J10.4 (Pin_4), J8.4 (Pin_4), J9.4 (Pin_4), Q2.3 (S), Q3.3 (S), Q4.3 (S), Q5.3 (S), Q6.3 (S), Q7.3 (S), R11.2, R14.2, R17.2, R20.2, R23.2, R26.2, R8.2
- net VDD: now also C14.1, C15.1, C16.1, J10.1 (Pin_1), J8.1 (Pin_1), J9.1 (Pin_1)
- net at R7.1: now also Q1.3 (S)
- net UART_2_RX: now reaches U1.1 (PB9)
- net UART_2_RX: now also J9.3 (Pin_3), R21.2
- net UART_2_TX: now reaches U1.12 (PA5)
- net UART_2_TX: now also J9.2 (Pin_2), R16.2
- net LED_SIG: now reaches U1.18 (PA8)
- net LED_SIG: now also R9.1
- net UART_1_TX: now reaches U1.19 (PA9)
- net UART_1_TX: now also J8.2 (Pin_2), R10.2
- net UART_1_RX: now reaches U1.21 (PA10)
- net UART_1_RX: now also J8.3 (Pin_3), R13.2
- net UART_3_TX: now reaches U1.7 (PA0)
- net UART_3_TX: now also J10.2 (Pin_2), R22.2
- net UART_3_RX: now reaches U1.8 (PA1)
- net UART_3_RX: now also J10.3 (Pin_3), R27.2
- new net: D7.2 (A), R25.2
- new net: D7.1 (K), Q7.1 (D)
- new net: D2.1 (K), Q2.1 (D)
- new net: Q2.2 (G), R10.1, R11.1
- new net: D5.1 (K), Q5.1 (D)
- new net: D5.2 (A), R19.2
- new net: Q4.2 (G), R16.1, R17.1
- new net: D6.2 (A), R24.2
- new net: Q1.2 (G), R8.1, R9.2
- new net: D3.2 (A), R15.2
- new net: D2.2 (A), R12.2
- new net: Q7.2 (G), R26.1, R27.1
- new net: Q3.2 (G), R13.1, R14.1
- new net: Q5.2 (G), R20.1, R21.1
- new net: D4.2 (A), R18.2
- new net: D3.1 (K), Q3.1 (D)
- new net: Q6.2 (G), R22.1, R23.1
- new net: D6.1 (K), Q6.1 (D)
- new net: D4.1 (K), Q4.1 (D)
- no-connect marks 2 -> 21
Other:
- note added: "ADD LEVEL SHIFTER RETURN + RETURN"
- note added: "LEDS DISPLAY"
- note added: "UART_1_LEDs"
- note added: "UART_2_LEDs"
- note added: "UART_3_LEDs"
- note added: "UARTs"
- moved on the sheet: C10, C11, C12, C13, C6, C7, C8, C9, D1, J2, J3, J4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

Commit message: [SMA] Edit schematic + Add footprints + begin PCB
Parts:
- removed C10, C11, C12, C9: TBD, Capacitor_SMD:C_0805_2012Metric_Pad1.18x1.45mm_HandSolder, symbol Device:C
- removed C13: TBD, Capacitor_SMD:CP_Elec_5x3, symbol Device:C_Polarized_US
- removed C14, C15, C16: C, symbol Device:C
- removed D1: TBD, symbol Device:D_Schottky
- removed L1: TBD, symbol Device:L
- removed Q1: Q_PMOS_DGS, symbol Device:Q_PMOS_DGS
- removed R2, R4, R5: TBD, Resistor_SMD:R_0805_2012Metric_Pad1.20x1.40mm_HandSolder, symbol Device:R
- removed R8: 10k, Resistor_SMD:R_0805_2012Metric_Pad1.20x1.40mm_HandSolder, symbol Device:R
- removed R9: 0, Resistor_SMD:R_0805_2012Metric_Pad1.20x1.40mm_HandSolder, symbol Device:R
- removed U3: TPS54331DR, PCM_Package_SO_AKL:TI_SO-PowerPAD-8_ThermalVias, symbol Regulator_Switching:TPS54331
- removed Y1: Crystal, symbol Device:Crystal
- added C1, C11: 100uF, Capacitor_THT:CP_Radial_D8.0mm_P3.50mm, symbol Device:C_Polarized_US
- added C17, C18: 0.1uF, Capacitor_SMD:C_0805_2012Metric_Pad1.18x1.45mm_HandSolder, symbol Device:C
- added C2: 4.7uF, Capacitor_SMD:C_0805_2012Metric_Pad1.18x1.45mm_HandSolder, symbol Device:C
- added C3: 100nF, Capacitor_SMD:C_0805_2012Metric_Pad1.18x1.45mm_HandSolder, symbol Device:C
- added C4, C5, C6: 22uF, Capacitor_SMD:C_0805_2012Metric_Pad1.18x1.45mm_HandSolder, symbol Device:C
- added C7: 1uF, Capacitor_SMD:C_0805_2012Metric_Pad1.18x1.45mm_HandSolder, symbol Device:C
- added H1, H2, H3: M2, MountingHole:MountingHole_2.7mm_M2.5_DIN965_Pad, symbol Mechanical:MountingHole_Pad
- added J14, J15, J16, J17, J18, J19: Conn_01x03_Female, Connector_JST:JST_XH_B3B-XH-A_1x03_P2.50mm_Vertical, symbol Connector:Conn_01x03_Female
- added J2: Conn_Alt_0, Connector_JST:JST_XH_B4B-XH-A_1x04_P2.50mm_Vertical, symbol Connector_Generic:Conn_01x04
- added J20, J21, J22, J23, J24, J25: Conn_01x03_Female, Connector_Wire:SolderWirePad_1x03_Corner_SMD, symbol Connector:Conn_01x03_Female
- added J27: SWD_TAG_Connector, Connector:Tag-Connect_TC2030-IDC-NL_2x03_P1.27mm_Vertical, symbol Connector_Generic:Conn_02x03_Odd_Even
- added J4: Conn_Alt_4, Connector_JST:JST_XH_B4B-XH-A_1x04_P2.50mm_Vertical, symbol Connector_Generic:Conn_01x04
- added J7: Conn_Alt_8, Connector_JST:JST_XH_B4B-XH-A_1x04_P2.50mm_Vertical, symbol Connector_Generic:Conn_01x04
- added R21: 10k, Resistor_SMD:R_0805_2012Metric_Pad1.20x1.40mm_HandSolder, symbol Device:R
- added R25: 0, Resistor_SMD:R_0805_2012Metric_Pad1.20x1.40mm_HandSolder, symbol Device:R
- added U1: TLVM23625RDNR, Package_DFN_QFN:QFN-FCMOD11_RDN_TEX, symbol Regulator_Linear:TLVM23625RDNR
- added U4: TXB0102DCU, Package_SO:VSSOP-8_2.4x2.1mm_P0.5mm, symbol Logic_LevelTranslator:TXB0102DCU
- added Y1: Crystal_GND24, Crystal:Crystal_SMD_2016-4Pin_2.0x1.6mm, symbol Device:Crystal_GND24
- C8: value TBD -> 100uF; footprint (none) -> Capacitor_THT:CP_Radial_D8.0mm_P3.50mm
- J1: renamed from J8; footprint (none) -> Connector:QFN_4-M0G
- J10: renamed from J4; footprint Connector_JST:JST_XH_B3B-XH-A_1x03_P2.50mm_Vertical -> Connector_PinSocket_2.54mm:PinSocket_1x03_P2.54mm_Vertical
- J11: renamed from J5; footprint Connector_JST:JST_XH_B3B-XH-A_1x03_P2.50mm_Vertical -> Connector_PinSocket_2.54mm:PinSocket_1x03_P2.54mm_Vertical
- J12: renamed from J6; footprint Connector_JST:JST_XH_B3B-XH-A_1x03_P2.50mm_Vertical -> Connector_PinSocket_2.54mm:PinSocket_1x03_P2.54mm_Vertical
- J13: renamed from J7; footprint Connector_JST:JST_XH_B3B-XH-A_1x03_P2.50mm_Vertical -> Connector_PinSocket_2.54mm:PinSocket_1x03_P2.54mm_Vertical
- J3: renamed from J9; footprint (none) -> Connector:QFN_4-M0G
- J5: renamed from J10; footprint (none) -> Connector:QFN_4-M0G
- J8: renamed from J2; footprint Connector_JST:JST_XH_B3B-XH-A_1x03_P2.50mm_Vertical -> Connector_PinSocket_2.54mm:PinSocket_1x03_P2.54mm_Vertical
- J9: renamed from J3; footprint Connector_JST:JST_XH_B3B-XH-A_1x03_P2.50mm_Vertical -> Connector_PinSocket_2.54mm:PinSocket_1x03_P2.54mm_Vertical
- Q1: renamed from Q2; footprint (none) -> PCM_Package_TO_SOT_SMD_AKL:SOT-23_Handsoldering
- Q2: renamed from Q3; footprint (none) -> PCM_Package_TO_SOT_SMD_AKL:SOT-23_Handsoldering
- Q3: renamed from Q4; footprint (none) -> PCM_Package_TO_SOT_SMD_AKL:SOT-23_Handsoldering
- Q4: renamed from Q5; footprint (none) -> PCM_Package_TO_SOT_SMD_AKL:SOT-23_Handsoldering
- Q5: renamed from Q6; footprint (none) -> PCM_Package_TO_SOT_SMD_AKL:SOT-23_Handsoldering
- Q6: renamed from Q7; footprint (none) -> PCM_Package_TO_SOT_SMD_AKL:SOT-23_Handsoldering
- R3: value TBD -> 40.2k
- R6: value TBD -> 10k
- SW1: footprint (none) -> Button_Switch_SMD:SW_Push_1P1T_NO_CK_KSC7xxJ
- renumbered C6 to C10, C4 to C12, C1 to C13, C2 to C14, C3 to C15, C5 to C16, C7 to C9, D2 to D1, D3 to D2, D4 to D3, D5 to D4, D6 to D5, D7 to D6, J1 to J6, R12 to R1, R19 to R10, R16 to R11, R21 to R12, R17 to R13, R20 to R14, R1 to R15, R24 to R16, R25 to R17, R7 to R18, R22 to R19, R15 to R2, R27 to R20, R26 to R24, R10 to R4, R13 to R5, R11 to R7, R14 to R8, R18 to R9, U1 to U2, U2 to U3
Connections:
- net +3V3: now also C18.1, J27.1 (Pin_1), R21.2, U4.3 (VCCA), U4.6 (OE)
- net +5V: now also R3.1, C17.1, C4.1, C5.1, C6.1, J14.1 (Pin_1), J15.1 (Pin_1), J16.1 (Pin_1), J17.1 (Pin_1), J18.1 (Pin_1), J19.1 (Pin_1), J20.1 (Pin_1), J21.1 (Pin_1), J22.1 (Pin_1), J23.1 (Pin_1), J24.1 (Pin_1), J25.1 (Pin_1), U1.4 (VOUT), U4.7 (VCCB)
- net GND: now also R6.2, C1.2, C11.2, C17.2, C18.2, C2.2, C3.2, C4.2, C5.2, C6.2, C7.2, H1.1, H2.1, H3.1, J14.3 (Pin_3), J15.3 (Pin_3), J16.3 (Pin_3), J17.3 (Pin_3), J18.3 (Pin_3), J19.3 (Pin_3), J2.4 (Pin_4), J20.3 (Pin_3), J21.3 (Pin_3), J22.3 (Pin_3), J23.3 (Pin_3), J24.3 (Pin_3), J25.3 (Pin_3), J27.5 (Pin_5), J4.4 (Pin_4), J7.4 (Pin_4), R21.1, U1. (GND), U4.2 (GND), Y1.2, Y1.4; no longer R6.1
- net LED_SIG: now also U4.5 (A1)
- net NRST: now also J27.3 (Pin_3)
- net OSC_IN: now also Y1.3
- net SWDCLK: now also J27.4 (Pin_4)
- net SWDIO: now also J27.2 (Pin_2)
- net UART_1_RX: now also J2.3 (Pin_3)
- net UART_1_TX: now also J2.2 (Pin_2)
- net UART_2_RX: now also J4.3 (Pin_3)
- net UART_2_TX: now also J4.2 (Pin_2)
- net UART_3_RX: now also J7.3 (Pin_3)
- net UART_3_TX: now also J7.2 (Pin_2)
- net VDD: now also C1.1, C11.1, C2.1, C3.1, J2.1 (Pin_1), J4.1 (Pin_1), J7.1 (Pin_1), U1.2 (EN), U1.3 (VIN); no longer R3.2
- net at R18.1: now also U4.8 (B1)
- net at J8.2 (Pin_2), R18.2: now also J14.2 (Pin_2), J20.2 (Pin_2)
- net at C16.2, R15.1: now also Y1.1
- net at J11.2 (Pin_2), J12.2 (Pin_2): now also J17.2 (Pin_2), J18.2 (Pin_2), J23.2 (Pin_2), J24.2 (Pin_2)
- net at J13.2 (Pin_2): now also J19.2 (Pin_2), J25.2 (Pin_2), R25.1
- net at J10.2 (Pin_2), J9.2 (Pin_2): now also J15.2 (Pin_2), J16.2 (Pin_2), J21.2 (Pin_2), J22.2 (Pin_2)
- net LED_RET: now reaches U2.17 (PB2)
- net LED_RET: now also U4.4 (A2)
- new net: C7.1, U1.11 (RT), U1.8 (VCC)
- new net: R25.2, U4.1 (B2)
- new net: U1.5 (SW), U1.6 (SW)
- new net: R3.2, R6.1, U1.9 (FB)
- no-connect marks 21 -> 22
Other:
- note added: "Mounting Holes"
- note added: "Optionnal"
- note removed: "ADD LEVEL SHIFTER RETURN + RETURN"
- moved on the sheet: C10, C9, J10, J11, J12, J13, J3, J5, J8, J9, R18, U3

Commit message: [SMA] Finish PCB
Connections:
- net GND: now also U1.10 (GND); no longer U1. (GND)
Changed lines of the file:
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@@
       (effects (font (size 1.27 1.27)) hide)
     )
-    (pin "")
     (pin "1")
+    (pin "10")
     (pin "11")
     (pin "2")

Commit message: [SMA] Fix many  bug
Connections:
- net UART_1_RX: now also U2.10 (PA3); no longer U2.21 (PA10)
- net UART_1_TX: now also U2.9 (PA2); no longer U2.19 (PA9)
- net UART_2_RX: now also U2.21 (PA10); no longer U2.1 (PB9)
- net UART_2_TX: now also U2.19 (PA9); no longer U2.12 (PA5)
- no-connect marks 22 -> 21
Changed lines of the file:
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@@
   (junction (at 302.26 31.75) (diameter 0) (color 0 0 0 0)
   )
-  (no_connect (at 48.895 83.185))
+  (no_connect (at 53.975 83.185))
   (no_connect (at 64.135 83.185))
   (no_connect (at 61.595 83.185))
+  (no_connect (at 51.435 83.185))
   (no_connect (at 81.915 60.325))
   (no_connect (at 61.595 27.305))
   (no_connect (at 59.055 83.185))
   (no_connect (at 81.915 52.705))
-  (no_connect (at 51.435 83.185))
   (no_connect (at 151.13 109.855))
   (no_connect (at 151.13 107.315))
-  (no_connect (at 46.355 83.185))
   (no_connect (at 48.895 27.305))
   (no_connect (at 180.975 108.585))
@@
     (effects (font (size 1.27 1.27)) (justify left bottom))
   )
-  (label "UART_1_TX" (at 81.915 62.865 0) (fields_autoplaced)
-    (effects (font (size 1.27 1.27)) (justify left bottom))
+  (label "UART_1_RX" (at 48.895 83.185 270) (fields_autoplaced)
+    (effects (font (size 1.27 1.27)) (justify right bottom))
   )
   (label "NRST" (at 31.115 62.865 180) (fields_autoplaced)
@@
     (effects (font (size 1.27 1.27)) (justify left bottom))
   )
+  (label "UART_1_TX" (at 46.355 83.185 270) (fields_autoplaced)
+    (effects (font (size 1.27 1.27)) (justify right bottom))
+  )
   (label "SWDCLK" (at 151.13 102.235 0) (fields_autoplaced)
     (effects (font (size 1.27 1.27)) (justify left bottom))
   )
-  (label "UART_1_RX" (at 81.915 57.785 0) (fields_autoplaced)
-    (effects (font (size 1.27 1.27)) (justify left bottom))
-  )
   (label "UART_2_RX" (at 297.18 67.945 180) (fields_autoplaced)
     (effects (font (size 1.27 1.27)) (justify right bottom))
   )
-  (label "UART_2_RX" (at 31.115 50.165 180) (fields_autoplaced)
-    (effects (font (size 1.27 1.27)) (justify right bottom))
-  )
-  (label "UART_2_TX" (at 53.975 83.185 270) (fields_autoplaced)
-    (effects (font (size 1.27 1.27)) (justify right bottom))
+  (label "UART_2_TX" (at 81.915 62.865 0) (fields_autoplaced)
+    (effects (font (size 1.27 1.27)) (justify left bottom))
+  )
+  (label "UART_2_RX" (at 81.915 57.785 0) (fields_autoplaced)
+    (effects (font (size 1.27 1.27)) (justify left bottom))
   )
   (label "UART_2_TX" (at 297.18 65.405 180) (fields_autoplaced)
