File: Small_Wall/Small_Wall.kicad_sch (KiCad schematic)
At the start: 29 parts, among them J1 Conn_01x03, J2 Conn_01x03, J4 Conn_01x03, J5 Conn_01x03, U1 IN-PI55TATPRPGPB, U2 IN-PI55TATPRPGPB, U3 IN-PI55TATPRPGPB, U4 IN-PI55TATPRPGPB, U5 IN-PI55TATPRPGPB, U6 IN-PI55TATPRPGPB, U7 IN-PI55TATPRPGPB

Commit message: [SMA][WALL] Update wall
Parts:
- removed C1, C7: 100nF, Capacitor_SMD:C_0805_2012Metric, symbol Device:C
- removed JP10, JP4: SolderJumper_2_Open, Jumper:SolderJumper-2_P1.3mm_Open_RoundedPad1.0x1.5mm, symbol Jumper:SolderJumper_2_Open
- removed U1, U7: IN-PI55TATPRPGPB, LED_SMD:IN-PI55TATPRPGPB, symbol LED:IN-PI55TATPRPGPB
- renumbered C2 to C1, C3 to C2, C4 to C3, C5 to C4, C6 to C5, J4 to J3, J5 to J4, JP5 to JP3, JP6 to JP4, JP7 to JP5, JP8 to JP6, JP9 to JP7, JP11 to JP8, JP12 to JP9, U2 to U1, U3 to U2, U4 to U3, U5 to U4, U6 to U5
Connections:
- net at JP1.2 (B), JP2.2 (B): now also JP3.1 (A), U1.4 (DIN)
- net at JP7.2 (B), U5.2 (DOUT): now also JP8.2 (B), JP9.2 (B)
